File: Shields 8.0/ShieldCatodoComun/ShieldCatodoComun.kicad_pcb (KiCad board)
At the start: 2 copper layers, 68.6 x 53.3 mm, 8 parts, among them J1 Power, J2 Digital/PWM, J3 Analog, J4 Digital/PWM

Commit message: Implementacion del PCB
Parts:
- added Q1: 2N2219, Package_TO_SOT_THT:TO-39-3, F.Cu at (107.5, 59.0)
- added Q2: 2N2219, Package_TO_SOT_THT:TO-39-3, F.Cu at (121.0, 59.0)
- added Q3: 2N2219, Package_TO_SOT_THT:TO-39-3, F.Cu at (141.5, 59.0)
- added R1: R, Resistor_THT:R_Axial_DIN0207_L6.3mm_D2.5mm_P10.16mm_Horizontal, F.Cu at (117.9, 93.7)
- added R10: R, Resistor_THT:R_Axial_DIN0207_L6.3mm_D2.5mm_P10.16mm_Horizontal, F.Cu at (154.4, 93.7)
- added R11: R, Resistor_THT:R_Axial_DIN0207_L6.3mm_D2.5mm_P10.16mm_Horizontal, F.Cu at (158.4, 93.7)
- added R2: R, Resistor_THT:R_Axial_DIN0207_L6.3mm_D2.5mm_P10.16mm_Horizontal, F.Cu at (122.0, 93.7)
- added R3: R, Resistor_THT:R_Axial_DIN0207_L6.3mm_D2.5mm_P10.16mm_Horizontal, F.Cu at (126.0, 93.7)
- added R4: R, Resistor_THT:R_Axial_DIN0207_L6.3mm_D2.5mm_P10.16mm_Horizontal, F.Cu at (130.1, 93.7)
- added R5: R, Resistor_THT:R_Axial_DIN0207_L6.3mm_D2.5mm_P10.16mm_Horizontal, F.Cu at (134.1, 93.7)
- added R6: R, Resistor_THT:R_Axial_DIN0207_L6.3mm_D2.5mm_P10.16mm_Horizontal, F.Cu at (138.2, 93.7)
- added R7: R, Resistor_THT:R_Axial_DIN0207_L6.3mm_D2.5mm_P10.16mm_Horizontal, F.Cu at (142.2, 93.7)
- added R8: R, Resistor_THT:R_Axial_DIN0207_L6.3mm_D2.5mm_P10.16mm_Horizontal, F.Cu at (146.3, 93.7)
- added R9: R, Resistor_THT:R_Axial_DIN0207_L6.3mm_D2.5mm_P10.16mm_Horizontal, F.Cu at (150.3, 93.7)
- added RV2: R_Potentiometer, Potentiometer_THT:Potentiometer_Alpha_RD901F-40-00D_Single_Vertical, F.Cu at (104.5, 82.2)
- added U1: D168K, Display_7Segment:D1X8K, F.Cu at (117.9, 79.1)
- added U2: D168K, Display_7Segment:D1X8K, F.Cu at (131.9, 79.1)
- added U3: D168K, Display_7Segment:D1X8K, F.Cu at (146.0, 79.1)
