File: Shields-8.0/ShieldCatodoComun/ShieldCatodoComun.kicad_sch (KiCad schematic)
At the start: 24 parts, among them J1 Power, J2 Digital/PWM, J3 Analog, J4 Digital/PWM, Q1 2N2219, Q2 2N2219, Q3 2N2219, U1 D168K, U2 D168K, U3 D168K

Commit message: Arreglos menores
Connections:
- net RX/0: now also J4.7 (Pin_7), JP1.1 (A); no longer J2.6 (Pin_6), JP1.3 (B)
- new net: J2.6 (Pin_6), JP1.3 (B)
Other:
- moved on the sheet: JP1, JP2
Changed lines of the file:
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@@
 	)
 	(junction
-		(at 69.85 90.17)
-		(diameter 0)
-		(color 0 0 0 0)
-	)
-	(junction
 		(at 246.38 95.25)
 		(diameter 0)
@@
 	(wire
 		(pts
-			(xy 66.04 41.91) (xy 66.04 83.82)
+			(xy 53.34 41.91) (xy 53.34 83.82)
 		)
 		(stroke
@@
 	(wire
 		(pts
-			(xy 66.04 114.3) (xy 68.58 114.3)
+			(xy 69.85 114.3) (xy 74.93 114.3)
 		)
 		(stroke
@@
 	(wire
 		(pts
-			(xy 69.85 90.17) (xy 69.85 39.37)
+			(xy 69.85 39.37) (xy 69.85 101.6)
 		)
 		(stroke
@@
 	(wire
 		(pts
-			(xy 66.04 101.6) (xy 66.04 100.33)
-		)
-		(stroke
-			(width 0)
-			(type default)
-		)
-	)
-	(wire
-		(pts
 			(xy 222.25 60.96) (xy 222.25 87.63)
 		)
@@
 	(wire
 		(pts
-			(xy 68.58 114.3) (xy 68.58 74.93)
+			(xy 74.93 114.3) (xy 74.93 74.93)
 		)
 		(stroke
@@
 	(wire
 		(pts
-			(xy 69.85 100.33) (xy 69.85 90.17)
-		)
-		(stroke
-			(width 0)
-			(type default)
-		)
-	)
-	(wire
-		(pts
 			(xy 185.42 59.69) (xy 220.98 59.69)
 		)
@@
 	(wire
 		(pts
-			(xy 66.04 99.06) (xy 66.04 96.52)
+			(xy 53.34 99.06) (xy 53.34 96.52)
 		)
 		(stroke
@@
 	(wire
 		(pts
-			(xy 69.85 90.17) (xy 73.66 90.17)
+			(xy 57.15 90.17) (xy 73.66 90.17)
 		)
 		(stroke
@@
 	(wire
 		(pts
-			(xy 69.85 107.95) (xy 76.2 107.95)
+			(xy 73.66 107.95) (xy 76.2 107.95)
 		)
 		(stroke
@@
 	(wire
 		(pts
-			(xy 66.04 100.33) (xy 69.85 100.33)
-		)
-		(stroke
-			(width 0)
-			(type default)
-		)
-	)
-	(wire
-		(pts
 			(xy 62.23 34.29) (xy 64.77 34.29)
 		)
@@
 	(wire
 		(pts
-			(xy 62.23 41.91) (xy 66.04 41.91)
+			(xy 53.34 41.91) (xy 62.23 41.91)
 		)
 		(stroke
@@
 	(wire
 		(pts
-			(xy 62.23 99.06) (xy 66.04 99.06)
+			(xy 53.34 99.06) (xy 62.23 99.06)
 		)
 		(stroke
@@
 	(wire
 		(pts
-			(xy 62.23 74.93) (xy 68.58 74.93)
+			(xy 62.23 74.93) (xy 74.93 74.93)
 		)
 		(stroke
@@
 	(symbol
 		(lib_id "Jumper:Jumper_3_Open")
-		(at 66.04 90.17 90)
+		(at 53.34 90.17 90)
 		(unit 1)
 		(exclude_from_sim yes)
@@
 		(fields_autoplaced yes)
 		(property "Reference" "JP2"
-			(at 63.5 88.8999 90)
+			(at 50.8 88.8999 90)
 			(effects
 				(font
@@
 		)
 		(property "Value" "Jumper_3_Open"
-			(at 63.5 91.4399 90)
+			(at 50.8 91.4399 90)
 			(effects
 				(font
@@
 		)
 		(property "Footprint" ""
-			(at 66.04 90.17 0)
+			(at 53.34 90.17 0)
 			(effects
 				(font
@@
 		)
 		(property "Datasheet" "~"
-			(at 66.04 90.17 0)
+			(at 53.34 90.17 0)
 			(effects
 				(font
@@
 		)
 		(property "Description" "Jumper, 3-pole, both open"
-			(at 66.04 90.17 0)
+			(at 53.34 90.17 0)
 			(effects
 				(font
@@
 	(symbol
 		(lib_id "Jumper:Jumper_3_Open")
-		(at 66.04 107.95 90)
+		(at 69.85 107.95 90)
 		(unit 1)
 		(exclude_from_sim yes)
@@
 		(fields_autoplaced yes)
 		(property "Reference" "JP1"
-			(at 63.5 106.6799 90)
+			(at 67.31 106.6799 90)
 			(effects
 				(font
@@
 		)
 		(property "Value" "Jumper_3_Open"
-			(at 63.5 109.2199 90)
+			(at 67.31 109.2199 90)
 			(effects
 				(font
@@
 		)
 		(property "Footprint" ""
-			(at 66.04 107.95 0)
+			(at 69.85 107.95 0)
 			(effects
 				(font
@@
 		)
 		(property "Datasheet" "~"
-			(at 66.04 107.95 0)
+			(at 69.85 107.95 0)
 			(effects
 				(font
@@
 		)
 		(property "Description" "Jumper, 3-pole, both open"
-			(at 66.04 107.95 0)
+			(at 69.85 107.95 0)
 			(effects
 				(font
