File: Shields-8.0/ShieldAnodoComun/ShieldAnodoComun.kicad_pcb (KiCad board)
At the start: 2 copper layers, 126.8 x 53.3 mm, 30 parts, among them J1 Power, J2 Digital/PWM, J3 Analog, J4 Digital/PWM, Q1 BC548, Q2 BC548, Q4 BC548, SW1 SW_Push, SW2 SW_Push, SW3 SW_Push, U1 HDSP-7501, U2 HDSP-7501, U4 HDSP-7501

Commit message: Arreglos para enrutar
Parts:
- RV2: footprint Potentiometer_THT:Potentiometer_Alpha_RD901F-40-00D_Single_Vertical -> Potentiometer_THT:Potentiometer_Alps_RK09K_Single_Horizontal
- U1, U2, U4: footprint Display_7Segment:D1X8K -> Display_Mod:D1X8K-comun-medio
- moved SW3 83.8 mm to (107.0, 90.5), turned to -90 degrees
- moved SW2 74.1 mm to (115.5, 90.5), turned to -90 degrees
- moved SW1 65.2 mm to (124.0, 90.5), turned to -90 degrees
- moved R14 43.9 mm to (157.8, 79.2), turned to -90 degrees
- moved R13 41.2 mm to (161.9, 79.2), turned to -90 degrees
- moved R12 39.0 mm to (165.9, 79.2), turned to -90 degrees
- moved R11 33.9 mm to (105.8, 52.2)
- moved R9 33.9 mm to (113.9, 52.2)
- moved R10 33.9 mm to (109.8, 52.2)
- moved Q3 32.6 mm to (102.9, 83.5)
- moved R1 32.4 mm to (153.3, 54.6), turned to -90 degrees
- moved Q2 31.8 mm to (102.9, 76.2)
- moved R8 28.0 mm to (124.9, 54.6), turned to -90 degrees
- moved R2 24.8 mm to (149.3, 54.6), turned to -90 degrees
- moved RV2 21.8 mm to (164.1, 71.9), turned to 180 degrees
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- renumbered Q4 to Q1, Q1 to Q2, Q2 to Q3
Connections:
- net Net-(J2-Pin_6) renamed /12
- net Net-(J2-Pin_7) renamed /*11
- net Net-(U1-A) renamed /R8
- net Net-(U1-B) renamed /R7
- net Net-(U1-F) renamed /R3
- R1 pad 1: /7 -> Net-(JP2-C)
- R1 pad 2: Net-(U1-DP) -> /R1
- R2 pad 1: /*6 -> Net-(JP1-C)
- R2 pad 2: Net-(U1-G) -> /R2
- R3 pad 1: /*5 -> /2
- R4 pad 1: /4 -> /*3
- R4 pad 2: Net-(U1-E) -> /R4
- R5 pad 1: /*3 -> /4
- R5 pad 2: Net-(U1-D) -> /R5
- R6 pad 1: /2 -> /*5
- R6 pad 2: Net-(U1-C) -> /R6
- R7 pad 1: Net-(JP1-C) -> /*6
- R8 pad 1: Net-(JP2-C) -> /7
- U1 pad 3: Net-(U1-G) -> /R4
- U1 pad 4: Net-(U1-E) -> /R2
- U1 pad 5: Net-(U1-D) -> /R1
- U1 pad 7: Net-(U1-DP) -> /R6
- U1 pad 8: Net-(U1-C) -> /R5
- U2 pad 3: Net-(U1-G) -> /R4
- U2 pad 4: Net-(U1-E) -> /R2
- U2 pad 5: Net-(U1-D) -> /R1
- U2 pad 7: Net-(U1-DP) -> /R6
- U2 pad 8: Net-(U1-C) -> /R5
- U4 pad 3: Net-(U1-G) -> /R4
- U4 pad 4: Net-(U1-E) -> /R2
- U4 pad 5: Net-(U1-D) -> /R1
- U4 pad 7: Net-(U1-DP) -> /R6
- U4 pad 8: Net-(U1-C) -> /R5
Routing:
- net Net-(U1-E): track 46.9 -> 0.00 mm
- net Net-(U1-G): track 46.2 -> 0.00 mm
- net /R3: track 45.9 -> 0.00 mm
- net Net-(U1-DP): track 45.4 -> 0.00 mm
- net Net-(U1-C): track 43.0 -> 0.00 mm
- net Net-(U1-D): track 42.2 -> 0.00 mm
- net /R7: track 41.4 -> 0.00 mm
- net /R8: track 39.3 -> 0.00 mm
- net /RX/0: track 6.13 -> 0.00 mm
- net Net-(J4-Pin_8): track 5.26 -> 0.28 mm
- net Net-(Q2-C): track 19.4 -> 15.2 mm
- net Net-(Q1-C): track 19.4 -> 15.2 mm
- net Net-(Q3-C): track 19.4 -> 15.2 mm
Other:
- board size 126.8 x 53.3 mm -> 68.6 x 53.3 mm

Commit message: Continuacion de enrutados
Parts:
- moved SW1 22.0 mm to (103.4, 98.0), turned to 90 degrees
- moved RV2 17.7 mm to (160.2, 89.2)
- moved SW3 13.8 mm to (118.6, 98.0), turned to 90 degrees
- moved R12 12.1 mm to (166.1, 67.1)
- moved R13 12.1 mm to (162.0, 67.1)
- moved R14 12.1 mm to (157.9, 67.1)
- moved SW2 8.70 mm to (111.0, 98.0), turned to 90 degrees
- moved Q3 5.28 mm to (108.1, 83.8)
- moved Q2 5.20 mm to (108.1, 76.2)
- moved Q1 5.18 mm to (108.1, 69.5)
- moved R11 2.94 mm to (107.6, 54.5)
- moved R1 2.84 mm to (153.3, 57.5)
- moved R2 2.84 mm to (149.3, 57.5)
- moved R3 2.84 mm to (145.2, 57.5)
- moved R4 2.84 mm to (141.2, 57.5)
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Connections:
- JP1 pad 3: /12 -> /*9
- JP2 pad 3: /*11 -> /*10
- R10 pad 1: /*9 -> /12
- R11 pad 1: /*10 -> /13
- R9 pad 1: /8 -> /*11
Routing:
- net /SDA/A4: track 0.00 -> 98.5 mm
- net GND: track 0.00 -> 89.5 mm
- net /SCL/A5: track 0.00 -> 89.4 mm
- net +5V: track 0.00 -> 84.8 mm
- net /R3: track 0.00 -> 84.5 mm, vias 0 -> 1
- net /A3: track 0.00 -> 81.4 mm, vias 0 -> 2
- net /R4: track 0.00 -> 79.6 mm
- net /*10: track 0.00 -> 64.7 mm
- net /*9: track 0.00 -> 62.5 mm
- net /R1: track 0.00 -> 57.6 mm
- net /R2: track 0.00 -> 57.4 mm, vias 0 -> 1
- net Net-(Q1-C): track 15.2 -> 60.9 mm, vias 0 -> 5
- net /R8: track 0.00 -> 39.5 mm
- net /R5: track 0.00 -> 38.0 mm
- net Net-(Q3-C): track 15.2 -> 49.6 mm, vias 0 -> 5
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