File: Shields-8.0/ShieldAnodoComun/ShieldAnodoComun.kicad_sch (KiCad schematic)
At the start: 30 parts, among them J1 Power, J2 Digital/PWM, J3 Analog, J4 Digital/PWM, Q1 BC548, Q2 BC548, Q4 BC548, SW1 SW_Push, SW2 SW_Push, SW3 SW_Push, U1 HDSP-7501, U2 HDSP-7501, U4 HDSP-7501

Commit message: Arreglos para enrutar
Parts:
- RV2: footprint Potentiometer_THT:Potentiometer_Alpha_RD901F-40-00D_Single_Vertical -> Potentiometer_THT:Potentiometer_Alps_RK09K_Single_Horizontal
- U1, U2, U4: footprint Display_7Segment:D1X8K -> Display_Mod:D1X8K-comun-medio
- renumbered Q4 to Q1, Q1 to Q2, Q2 to Q3
Connections:
- net *11: now also J2.7 (Pin_7), JP2.3 (B)
- net *3: now also R4.1; no longer R5.1
- net *5: now also R6.1; no longer R3.1
- net *6: now also R7.1; no longer R2.1
- net 12: now also J2.6 (Pin_6), JP1.3 (B)
- net 2: now also R3.1; no longer R6.1
- net 4: now also R5.1; no longer R4.1
- net 7: now also R8.1; no longer R1.1
- net RX/0: no longer JP2.2 (C), R8.1
- net R2: now reaches U1.4 (E), U2.4 (E), U4.4 (E)
- net R2: now also R2.2; no longer R4.2
- net R3: now reaches R3.2, U1.2 (F), U2.2 (F), U4.2 (F)
- net at JP1.2 (C): now also R2.1; no longer R7.1
- net R7: now reaches R7.2, U1.9 (B), U2.9 (B), U4.9 (B)
- net R8: now reaches R8.2, U1.10 (A), U2.10 (A), U4.10 (A)
- net R5: now reaches U1.8 (C), U2.8 (C), U4.8 (C)
- net R5: now also R5.2; no longer R6.2
- net R4: now reaches U1.3 (G), U2.3 (G), U4.3 (G)
- net R4: now also R4.2; no longer R2.2
- net R1: now reaches U1.5 (D), U2.5 (D), U4.5 (D)
- net R1: now also R1.2; no longer R5.2
- net R6: now reaches U1.7 (DP), U2.7 (DP), U4.7 (DP)
- net R6: now also R6.2; no longer R1.2
- new net: JP2.2 (C), R1.1
Other:
- moved on the sheet: JP2, R1, R2, R3, R4, R5, R6, R7, R8

Commit message: Continuacion de enrutados
Connections:
- net *10: now also JP2.3 (B); no longer R11.1
- net *11: now also R9.1; no longer JP2.3 (B)
- net *9: now also JP1.3 (B); no longer R10.1
- net 12: now also R10.1; no longer JP1.3 (B)
- net 13: now also R11.1
- net 8: no longer R9.1
Changed lines of the file:
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@@
 	)
 	(junction
-		(at 67.31 41.91)
+		(at 67.31 44.45)
 		(diameter 0)
 		(color 0 0 0 0)
@@
 	)
 	(junction
-		(at 69.85 39.37)
+		(at 69.85 46.99)
 		(diameter 0)
 		(color 0 0 0 0)
@@
 	(wire
 		(pts
-			(xy 62.23 44.45) (xy 90.17 44.45)
-		)
-		(stroke
-			(width 0)
-			(type solid)
-		)
-	)
-	(wire
-		(pts
 			(xy 224.79 82.55) (xy 228.6 82.55)
 		)
@@
 	(wire
 		(pts
-			(xy 74.93 41.91) (xy 67.31 41.91)
-		)
-		(stroke
-			(width 0)
-			(type default)
-		)
-	)
-	(wire
-		(pts
 			(xy 19.05 95.25) (xy 19.05 105.41)
 		)
@@
 	(wire
 		(pts
+			(xy 69.85 46.99) (xy 74.93 46.99)
+		)
+		(stroke
+			(width 0)
+			(type default)
+		)
+	)
+	(wire
+		(pts
 			(xy 44.45 120.65) (xy 44.45 133.35)
 		)
@@
 	(wire
 		(pts
+			(xy 67.31 44.45) (xy 74.93 44.45)
+		)
+		(stroke
+			(width 0)
+			(type default)
+		)
+	)
+	(wire
+		(pts
 			(xy 199.39 113.03) (xy 201.93 113.03)
 		)
@@
 	(wire
 		(pts
-			(xy 67.31 88.9) (xy 53.34 88.9)
-		)
-		(stroke
-			(width 0)
-			(type default)
-		)
-	)
-	(wire
-		(pts
 			(xy 31.75 39.37) (xy 34.29 39.37)
 		)
@@
 	(wire
 		(pts
-			(xy 62.23 36.83) (xy 74.93 36.83)
+			(xy 62.23 36.83) (xy 90.17 36.83)
 		)
 		(stroke
@@
 	(wire
 		(pts
-			(xy 62.23 39.37) (xy 69.85 39.37)
+			(xy 62.23 39.37) (xy 88.9 39.37)
 		)
 		(stroke
@@
 	(wire
 		(pts
+			(xy 62.23 46.99) (xy 69.85 46.99)
+		)
+		(stroke
+			(width 0)
+			(type default)
+		)
+	)
+	(wire
+		(pts
 			(xy 62.23 62.23) (xy 82.55 62.23)
 		)
@@
 	(wire
 		(pts
-			(xy 62.23 46.99) (xy 88.9 46.99)
-		)
-		(stroke
-			(width 0)
-			(type solid)
-		)
-	)
-	(wire
-		(pts
 			(xy 24.13 110.49) (xy 16.51 110.49)
 		)
@@
 	(wire
 		(pts
-			(xy 69.85 39.37) (xy 69.85 101.6)
-		)
-		(stroke
-			(width 0)
-			(type default)
-		)
-	)
-	(wire
-		(pts
 			(xy 179.07 123.19) (xy 209.55 123.19)
 		)
@@
 	(wire
 		(pts
+			(xy 53.34 88.9) (xy 67.31 88.9)
+		)
+		(stroke
+			(width 0)
+			(type default)
+		)
+	)
+	(wire
+		(pts
 			(xy 222.25 60.96) (xy 222.25 87.63)
 		)
@@
 	(wire
 		(pts
-			(xy 87.63 113.03) (xy 87.63 49.53)
-		)
-		(stroke
-			(width 0)
-			(type default)
-		)
-	)
-	(wire
-		(pts
 			(xy 148.59 95.25) (xy 160.02 95.25)
 		)
@@
 	(wire
 		(pts
+			(xy 90.17 36.83) (xy 90.17 104.14)
+		)
+		(stroke
+			(width 0)
+			(type default)
+		)
+	)
+	(wire
+		(pts
 			(xy 191.77 113.03) (xy 190.5 113.03)
 		)
@@
 	(wire
 		(pts
-			(xy 67.31 41.91) (xy 62.23 41.91)
+			(xy 69.85 46.99) (xy 69.85 101.6)
+		)
+		(stroke
+			(width 0)
+			(type default)
+		)
+	)
+	(wire
+		(pts
+			(xy 62.23 41.91) (xy 87.63 41.91)
 		)
 		(stroke
@@
 	(wire
 		(pts
-			(xy 67.31 41.91) (xy 67.31 88.9)
+			(xy 67.31 44.45) (xy 67.31 88.9)
 		)
 		(stroke
@@
 	(wire
 		(pts
-			(xy 74.93 39.37) (xy 69.85 39.37)
+			(xy 62.23 49.53) (xy 74.93 49.53)
 		)
 		(stroke
@@
 	(wire
 		(pts
-			(xy 88.9 105.41) (xy 88.9 46.99)
+			(xy 88.9 39.37) (xy 88.9 105.41)
 		)
 		(stroke
@@
 	(wire
 		(pts
+			(xy 87.63 41.91) (xy 87.63 113.03)
+		)
+		(stroke
+			(width 0)
+			(type default)
+		)
+	)
+	(wire
+		(pts
 			(xy 157.48 66.04) (xy 157.48 77.47)
 		)
@@
 	(wire
 		(pts
+			(xy 62.23 44.45) (xy 67.31 44.45)
+		)
+		(stroke
+			(width 0)
+			(type default)
+		)
+	)
+	(wire
+		(pts
 			(xy 228.6 113.03) (xy 227.33 113.03)
 		)
@@
 	(wire
 		(pts
-			(xy 90.17 104.14) (xy 90.17 44.45)
-		)
-		(stroke
-			(width 0)
-			(type default)
-		)
-	)
-	(wire
-		(pts
 			(xy 218.44 95.25) (xy 228.6 95.25)
 		)
@@
 		)
 	)
-	(wire
-		(pts
-			(xy 62.23 49.53) (xy 87.63 49.53)
-		)
-		(stroke
-			(width 0)
-			(type solid)
-		)
-	)
